Commit message: generated new usd files with paths pointing to local urdf files, removed iiwa14 files

File: robot/urdf/iiwa7.urdf (robot description, URDF)
Before this commit: robot iiwa7, 10 links, 9 joints
Links:
- link iiwa_link_0: geometry collision mesh filename=/home/david/bachelors-thesis/robot/meshes/iiwa7/collision/l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; visual mesh filename=/home/david/bachelors-thesis/robot/meshes/iiwa7/visual/link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
- link iiwa_link_1: geometry collision mesh filename=/home/david/bachelors-thesis/robot/meshes/iiwa7/collision/l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; visual mesh filename=/home/david/bachelors-thesis/robot/meshes/iiwa7/visual/link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
- link iiwa_link_2: geometry collision mesh filename=/home/david/bachelors-thesis/robot/meshes/iiwa7/collision/l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; visual mesh filename=/home/david/bachelors-thesis/robot/meshes/iiwa7/visual/link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
- link iiwa_link_3: geometry collision mesh filename=/home/david/bachelors-thesis/robot/meshes/iiwa7/collision/l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; visual mesh filename=/home/david/bachelors-thesis/robot/meshes/iiwa7/visual/link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
- link iiwa_link_4: geometry collision mesh filename=/home/david/bachelors-thesis/robot/meshes/iiwa7/collision/l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; visual mesh filename=/home/david/bachelors-thesis/robot/meshes/iiwa7/visual/link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
- link iiwa_link_5: geometry collision mesh filename=/home/david/bachelors-thesis/robot/meshes/iiwa7/collision/l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; visual mesh filename=/home/david/bachelors-thesis/robot/meshes/iiwa7/visual/link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
- link iiwa_link_6: geometry collision mesh filename=/home/david/bachelors-thesis/robot/meshes/iiwa7/collision/l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; visual mesh filename=/home/david/bachelors-thesis/robot/meshes/iiwa7/visual/link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
- link iiwa_link_7: geometry collision mesh filename=/home/david/bachelors-thesis/robot/meshes/iiwa7/collision/l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; visual mesh filename=/home/david/bachelors-thesis/robot/meshes/iiwa7/visual/link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
