Commit message: added gripper along with scripts for converting to urdf to usd and applying friction to gripper fingers

File: code/ros2_ws/src/kmr_iiwa_description/xacro/kmr_iiwa.urdf.xacro (robot description, xacro)
@@ -4,4 +4,5 @@
        so we don't include it again here (avoids duplicate <material> tags). -->
   <xacro:include filename="kmr_base.xacro"/>
+  <xacro:include filename="gripper.xacro"/>
   <xacro:include filename="iiwa7.xacro"/>
   <xacro:arg name="hardware_interface" default="PositionJointInterface"/>
@@ -20,3 +21,6 @@
     <origin xyz="${iiwa_mount_x} ${iiwa_mount_y} ${iiwa_mount_z}" rpy="0 0 0"/>
   </xacro:iiwa7>
+  <xacro:kmr_gripper parent="iiwa_link_ee" mesh_path="../meshes/gripper">
+    <origin xyz="0 0 0" rpy="0 0 0"/>
+  </xacro:kmr_gripper>
 </robot>
