Commit message: rotated revolute door handle, added april tags to door and handles

File: code/ros2_ws/src/kmr_iiwa_description/urdf/revolute_door.urdf (robot description, URDF)
Before this commit: robot revolute_door, 4 links, 3 joints
Links:
- added link door_tag_center; visual box size=0.08 0.08 0.001
- added link handle_tag_a; visual box size=0.025 0.025 0.001
- added link handle_tag_b; visual box size=0.025 0.025 0.001
- link handle_lever: mass 0.2 -> 0.25; geometry collision cylinder length=0.16 radius=0.014; visual cylinder length=0.16 radius=0.014
Joints:
- added joint door_tag_center_joint: type fixed, parent door_leaf, child door_tag_center, origin xyz=0.021 0.425 1.0 rpy=0 1.5708 0
- added joint handle_tag_a_joint: type fixed, parent handle_lever, child handle_tag_a, origin xyz=0.016 -0.015 0 rpy=0 1.5708 0
- added joint handle_tag_b_joint: type fixed, parent handle_lever, child handle_tag_b, origin xyz=0.016 -0.145 0 rpy=0 1.5708 0

File: code/ros2_ws/src/kmr_iiwa_description/urdf/sliding_door.urdf (robot description, URDF)
Before this commit: robot sliding_door, 3 links, 2 joints
Links:
- added link door_tag_center; visual box size=0.08 0.08 0.001
- added link handle_tag_a; visual box size=0.025 0.025 0.001
- added link handle_tag_b; visual box size=0.025 0.025 0.001
Joints:
- added joint door_tag_center_joint: type fixed, parent door_leaf, child door_tag_center, origin xyz=0.021 0.425 1.0 rpy=0 1.5708 0
- added joint handle_tag_a_joint: type fixed, parent handle, child handle_tag_a, origin xyz=0.086 0 -0.11 rpy=0 1.5708 0
- added joint handle_tag_b_joint: type fixed, parent handle, child handle_tag_b, origin xyz=0.086 0 0.11 rpy=0 1.5708 0

Commit message: added apriltags images to doors, replaced box with mesh

File: code/ros2_ws/src/kmr_iiwa_description/urdf/revolute_door.urdf (robot description, URDF)
Before this commit: robot revolute_door, 7 links, 6 joints
Links:
- link door_tag_center: mass None -> 0.001; geometry visual mesh filename=../meshes/tags/tag_quad.obj scale=0.08 0.08 1
- link handle_tag_a: mass None -> 0.001; geometry visual mesh filename=../meshes/tags/tag_quad.obj scale=0.025 0.025 1
- link handle_tag_b: mass None -> 0.001; geometry visual mesh filename=../meshes/tags/tag_quad.obj scale=0.025 0.025 1

File: code/ros2_ws/src/kmr_iiwa_description/urdf/sliding_door.urdf (robot description, URDF)
Before this commit: robot sliding_door, 6 links, 5 joints
Links:
- link door_tag_center: mass None -> 0.001; geometry visual mesh filename=../meshes/tags/tag_quad.obj scale=0.08 0.08 1
- link handle_tag_a: mass None -> 0.001; geometry visual mesh filename=../meshes/tags/tag_quad.obj scale=0.025 0.025 1
- link handle_tag_b: mass None -> 0.001; geometry visual mesh filename=../meshes/tags/tag_quad.obj scale=0.025 0.025 1

Commit message: optimized door urdf-s for working with rl

File: code/ros2_ws/src/kmr_iiwa_description/urdf/revolute_door.urdf (robot description, URDF)
Before this commit: robot revolute_door, 7 links, 6 joints
Joints:
- joint latch_joint: axis 1 0 0 -> (none); limit lower=0.0 upper=0.7 effort=20 velocity=3.0 -> (none); type revolute -> fixed
