Commit message: added camera and mount to robot

File: code/ros2_ws/src/kmr_iiwa_description/urdf/kmr_iiwa_full.urdf (robot description, URDF)
Before this commit: robot kmr_iiwa, 16 links, 15 joints
Links:
- added link camera_color_optical_frame
- added link camera_link, mass 0.072; collision box size=0.025 0.090 0.025; visual mesh filename=../meshes/camera/D435.stl
- added link camera_mount_link, mass 0.1929; collision box size=0.17774 0.17774 0.015; collision cylinder length=0.010 radius=0.003
Joints:
- added joint camera_color_optical_joint: type fixed, parent camera_link, child camera_color_optical_frame, origin xyz=0 0 0 rpy=-1.5707963267948966 0 -1.5707963267948966
- added joint camera_joint: type fixed, parent camera_mount_link, child camera_link, origin xyz=0 0 0.025 rpy=0 0 0
- added joint camera_mount_joint: type fixed, parent base_link, child camera_mount_link, origin xyz=0.363 0.184 0.7 rpy=0 0 0

File: code/ros2_ws/src/kmr_iiwa_description/xacro/kmr_iiwa.urdf.xacro (robot description, xacro)
@@ -5,4 +5,5 @@
   <xacro:include filename="kmr_base.xacro"/>
   <xacro:include filename="gripper.xacro"/>
+  <xacro:include filename="camera_mount.xacro"/>
   <xacro:include filename="iiwa7.xacro"/>
   <xacro:arg name="hardware_interface" default="PositionJointInterface"/>
@@ -24,3 +25,9 @@
     <origin xyz="0 0 0" rpy="0 0 0"/>
   </xacro:kmr_gripper>
+  <xacro:property name="camera_mount_x" value="0.363"/>
+  <xacro:property name="camera_mount_y" value="0.184"/>
+  <xacro:property name="camera_mount_z" value="${kmr_height}"/>
+  <xacro:kmr_camera_mount parent="base_link" mesh_path="../meshes/camera">
+    <origin xyz="${camera_mount_x} ${camera_mount_y} ${camera_mount_z}" rpy="0 0 0"/>
+  </xacro:kmr_camera_mount>
 </robot>

Commit message: added camera to urdf and py script to connect sim camera to ros2

File: code/ros2_ws/src/kmr_iiwa_description/urdf/kmr_iiwa_full.urdf (robot description, URDF)
Before this commit: robot kmr_iiwa, 19 links, 18 joints
Links:
- link camera_color_optical_frame: mass None -> 0.001
- link gripper_tcp: mass None -> 0.001
- link iiwa_link_ee: mass None -> 0.001

Commit message: implemented ros2_control for moving iiwa arm

File: code/ros2_ws/src/kmr_iiwa_description/urdf/kmr_iiwa_full.urdf (robot description, URDF)
Before this commit: robot kmr_iiwa, 19 links, 18 joints
Links:
- link camera_color_optical_frame: mass 0.001 -> None
- link gripper_tcp: mass 0.001 -> None
- link iiwa_link_ee: mass 0.001 -> None

File: code/ros2_ws/src/kmr_iiwa_description/xacro/kmr_iiwa.urdf.xacro (robot description, xacro)
@@ -7,4 +7,5 @@
   <xacro:include filename="camera_mount.xacro"/>
   <xacro:include filename="iiwa7.xacro"/>
+  <xacro:include filename="kmr_iiwa_ros2_control.xacro"/>
   <xacro:arg name="hardware_interface" default="PositionJointInterface"/>
   <xacro:arg name="robot_name" default="iiwa"/>
@@ -31,3 +32,6 @@
     <origin xyz="${camera_mount_x} ${camera_mount_y} ${camera_mount_z}" rpy="0 0 0"/>
   </xacro:kmr_camera_mount>
+  <xacro:kmr_iiwa_ros2_control
+      commands_topic="/isaac_joint_commands"
+      states_topic="/isaac_joint_states"/>
 </robot>

Commit message: changed mesh paths from relative paths to package-relative paths

File: code/ros2_ws/src/kmr_iiwa_description/urdf/kmr_iiwa_full.urdf (robot description, URDF)
Before this commit: robot kmr_iiwa, 19 links, 18 joints
Links:
- link base_link: geometry collision box size=1.08 0.63 0.7; visual mesh filename=package://kmr_iiwa_description/meshes/kmr_base/kmr_base_bod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 scale=1 1 1
- link camera_link: geometry collision box size=0.025 0.090 0.025; visual mesh filename=package://kmr_iiwa_description/meshes/camera/D435.stl
- link camera_mount_link: geometry collision box size=0.17774 0.17774 0.015; collision cylinder length=0.010 radius=0.003
- link gripper_base: geometry collision box size=0.085 0.085 0.020; collision cylinder length=0.015 radius=0.0315
- link gripper_finger_1: geometry collision mesh filename=package://kmr_iiwa_description/meshes/gripper/gripper_finge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; visual mesh filename=package://kmr_iiwa_description/meshes/gripper/gripper_finge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
- link gripper_finger_2: geometry collision mesh filename=package://kmr_iiwa_description/meshes/gripper/gripper_finge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; visual mesh filename=package://kmr_iiwa_description/meshes/gripper/gripper_finge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
- link gripper_finger_3: geometry collision mesh filename=package://kmr_iiwa_description/meshes/gripper/gripper_finge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; visual mesh filename=package://kmr_iiwa_description/meshes/gripper/gripper_finge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
- link gripper_finger_4: geometry collision mesh filename=package://kmr_iiwa_description/meshes/gripper/gripper_finge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; visual mesh filename=package://kmr_iiwa_description/meshes/gripper/gripper_finge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
- link iiwa_link_0: geometry collision mesh filename=package://kmr_iiwa_description/meshes/iiwa7/collision/link_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; visual mesh filename=package://kmr_iiwa_description/meshes/iiwa7/visual/link_0.s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
- link iiwa_link_1: geometry collision mesh filename=package://kmr_iiwa_description/meshes/iiwa7/collision/link_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; visual mesh filename=package://kmr_iiwa_description/meshes/iiwa7/visual/link_1.s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
- link iiwa_link_2: geometry collision mesh filename=package://kmr_iiwa_description/meshes/iiwa7/collision/link_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; visual mesh filename=package://kmr_iiwa_description/meshes/iiwa7/visual/link_2.s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
- link iiwa_link_3: geometry collision mesh filename=package://kmr_iiwa_description/meshes/iiwa7/collision/link_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; visual mesh filename=package://kmr_iiwa_description/meshes/iiwa7/visual/link_3.s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
- link iiwa_link_4: geometry collision mesh filename=package://kmr_iiwa_description/meshes/iiwa7/collision/link_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; visual mesh filename=package://kmr_iiwa_description/meshes/iiwa7/visual/link_4.s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
- link iiwa_link_5: geometry collision mesh filename=package://kmr_iiwa_description/meshes/iiwa7/collision/link_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; visual mesh filename=package://kmr_iiwa_description/meshes/iiwa7/visual/link_5.s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
- link iiwa_link_6: geometry collision mesh filename=package://kmr_iiwa_description/meshes/iiwa7/collision/link_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; visual mesh filename=package://kmr_iiwa_description/meshes/iiwa7/visual/link_6.s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
- link iiwa_link_7: geometry collision mesh filename=package://kmr_iiwa_description/meshes/iiwa7/collision/link_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; visual mesh filename=package://kmr_iiwa_description/meshes/iiwa7/visual/link_7.s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

File: code/ros2_ws/src/kmr_iiwa_description/xacro/camera_mount.xacro (robot description, xacro)
@@ -28,15 +28,6 @@
     - masa = 72g (Intel D400 datasheet, potvrđeno), inercija = box aprox.
       (90x25x25mm) — dovoljno precizno, kamera je zanemarive mase naspram
-      mounta/ruke (vidi handoff dok. §4).
-    - ⚠️ PLACEHOLDER: `camera_boss_top_z` (visina vrha bossa iznad ravnine
-      4 rupe) i pretpostavka da kamera sjedi FLAT (0° tilt, tripod-hole
-      centriran na os bossa, gleda +X) — potvrđeno FOV proračunom da radi
-      za ciljani raspon detekcije 1.0-1.5m (RGB V-FOV=42.5°, margina
-      4.6-9.9°). Kad popraviš boss, samo update-aj `camera_boss_top_z`.
-    - ⚠️ Nisam potvrdio koji kraj Z-osi mesha D435.stl je "prednji" (lens)
-      strana — pretpostavljam standardnu orijentaciju (dugi rub = lijevo-
-      desno baseline, kratki rub = naprijed-natrag). Provjeri vizualno u
-      SolidWorxu prije finalne montaže, ili mi reci pa ću ispraviti rpy.
-  camera_color_optical_frame — TF konvencija po §5 handoff dokumenta:
+      mounta/ruke.
+  camera_color_optical_frame — TF konvencija:
     body (X naprijed, Z gore) -> optical (Z naprijed, X desno, Y dolje),
     fiksna rotacija (-90°, 0°, -90°). Standardna realsense-ros konvencija.
@@ -53,5 +44,4 @@
       <color rgba="0.05 0.05 0.06 1.0"/>
     </material>
-    <!-- ⚠️ PLACEHOLDER dok se boss ne poveća za navoj (vidi header) -->
     <xacro:property name="camera_boss_top_z" value="0.025"/>
     <!-- ================= X-NOSAČ (camera_mount_link) ================= -->
@@ -124,5 +114,4 @@
       <child link="camera_link"/>
     </joint>
-    <!-- ================= OPTICAL FRAME (§5 handoff dokumenta) ================= -->
     <link name="camera_color_optical_frame"/>
     <joint name="camera_color_optical_joint" type="fixed">

File: code/ros2_ws/src/kmr_iiwa_description/xacro/iiwa7.xacro (robot description, xacro)
@@ -29,12 +29,12 @@
         <origin xyz="0 0 0" rpy="0 0 0"/>
         <geometry>
-          <mesh filename="../meshes/iiwa7/visual/link_0.stl"/>
-        </geometry>
-        <material name="Grey"/>
-      </visual>
-      <collision>
-        <origin xyz="0 0 0" rpy="0 0 0"/>
-        <geometry>
-          <mesh filename="../meshes/iiwa7/collision/link_0.stl"/>
+          <mesh filename="package://kmr_iiwa_description/meshes/iiwa7/visual/link_0.stl"/>
+        </geometry>
+        <material name="Grey"/>
+      </visual>
+      <collision>
+        <origin xyz="0 0 0" rpy="0 0 0"/>
+        <geometry>
+          <mesh filename="package://kmr_iiwa_description/meshes/iiwa7/collision/link_0.stl"/>
         </geometry>
         <material name="Grey"/>
@@ -70,5 +70,5 @@
         <origin xyz="0 0 0.0075" rpy="0 0 0"/>
         <geometry>
-          <mesh filename="../meshes/iiwa7/visual/link_1.stl"/>
+          <mesh filename="package://kmr_iiwa_description/meshes/iiwa7/visual/link_1.stl"/>
         </geometry>
         <material name="Orange"/>
@@ -77,5 +77,5 @@
         <origin xyz="0 0 0.0075" rpy="0 0 0"/>
         <geometry>
-          <mesh filename="../meshes/iiwa7/collision/link_1.stl"/>
+          <mesh filename="package://kmr_iiwa_description/meshes/iiwa7/collision/link_1.stl"/>
         </geometry>
         <material name="Orange"/>
@@ -104,12 +104,12 @@
         <origin xyz="0 0 0" rpy="0 0 0"/>
         <geometry>
-          <mesh filename="../meshes/iiwa7/visual/link_2.stl"/>
-        </geometry>
-        <material name="Orange"/>
-      </visual>
-      <collision>
-        <origin xyz="0 0 0" rpy="0 0 0"/>
-        <geometry>
-          <mesh filename="../meshes/iiwa7/collision/link_2.stl"/>
+          <mesh filename="package://kmr_iiwa_description/meshes/iiwa7/visual/link_2.stl"/>
+        </geometry>
+        <material name="Orange"/>
+      </visual>
+      <collision>
+        <origin xyz="0 0 0" rpy="0 0 0"/>
+        <geometry>
+          <mesh filename="package://kmr_iiwa_description/meshes/iiwa7/collision/link_2.stl"/>
         </geometry>
         <material name="Orange"/>
@@ -138,12 +138,12 @@
         <origin xyz="0 0 -0.026" rpy="0 0 0"/>
         <geometry>
-          <mesh filename="../meshes/iiwa7/visual/link_3.stl"/>
-        </geometry>
-        <material name="Orange"/>
-      </visual>
-      <collision>
-        <origin xyz="0 0 -0.026" rpy="0 0 0"/>
-        <geometry>
-          <mesh filename="../meshes/iiwa7/collision/link_3.stl"/>
+          <mesh filename="package://kmr_iiwa_description/meshes/iiwa7/visual/link_3.stl"/>
+        </geometry>
+        <material name="Orange"/>
+      </visual>
+      <collision>
+        <origin xyz="0 0 -0.026" rpy="0 0 0"/>
+        <geometry>
+          <mesh filename="package://kmr_iiwa_description/meshes/iiwa7/collision/link_3.stl"/>
         </geometry>
         <material name="Orange"/>
@@ -172,12 +172,12 @@
         <origin xyz="0 0 0" rpy="0 0 0"/>
         <geometry>
-          <mesh filename="../meshes/iiwa7/visual/link_4.stl"/>
-        </geometry>
-        <material name="Orange"/>
-      </visual>
-      <collision>
-        <origin xyz="0 0 0" rpy="0 0 0"/>
-        <geometry>
-          <mesh filename="../meshes/iiwa7/collision/link_4.stl"/>
+          <mesh filename="package://kmr_iiwa_description/meshes/iiwa7/visual/link_4.stl"/>
+        </geometry>
+        <material name="Orange"/>
+      </visual>
+      <collision>
+        <origin xyz="0 0 0" rpy="0 0 0"/>
+        <geometry>
+          <mesh filename="package://kmr_iiwa_description/meshes/iiwa7/collision/link_4.stl"/>
         </geometry>
         <material name="Orange"/>
@@ -206,12 +206,12 @@
         <origin xyz="0 0 -0.026" rpy="0 0 0"/>
         <geometry>
-          <mesh filename="../meshes/iiwa7/visual/link_5.stl"/>
-        </geometry>
-        <material name="Orange"/>
-      </visual>
-      <collision>
-        <origin xyz="0 0 -0.026" rpy="0 0 0"/>
-        <geometry>
-          <mesh filename="../meshes/iiwa7/collision/link_5.stl"/>
+          <mesh filename="package://kmr_iiwa_description/meshes/iiwa7/visual/link_5.stl"/>
+        </geometry>
+        <material name="Orange"/>
+      </visual>
+      <collision>
+        <origin xyz="0 0 -0.026" rpy="0 0 0"/>
+        <geometry>
+          <mesh filename="package://kmr_iiwa_description/meshes/iiwa7/collision/link_5.stl"/>
         </geometry>
         <material name="Orange"/>
@@ -240,12 +240,12 @@
         <origin xyz="0 0 0" rpy="0 0 0"/>
         <geometry>
-          <mesh filename="../meshes/iiwa7/visual/link_6.stl"/>
-        </geometry>
-        <material name="Orange"/>
-      </visual>
-      <collision>
-        <origin xyz="0 0 0" rpy="0 0 0"/>
-        <geometry>
-          <mesh filename="../meshes/iiwa7/collision/link_6.stl"/>
+          <mesh filename="package://kmr_iiwa_description/meshes/iiwa7/visual/link_6.stl"/>
+        </geometry>
+        <material name="Orange"/>
+      </visual>
+      <collision>
+        <origin xyz="0 0 0" rpy="0 0 0"/>
+        <geometry>
+          <mesh filename="package://kmr_iiwa_description/meshes/iiwa7/collision/link_6.stl"/>
         </geometry>
         <material name="Orange"/>
@@ -274,5 +274,5 @@
         <origin xyz="0 0 -0.0005" rpy="0 0 0"/>
         <geometry>
-          <mesh filename="../meshes/iiwa7/visual/link_7.stl"/>
+          <mesh filename="package://kmr_iiwa_description/meshes/iiwa7/visual/link_7.stl"/>
         </geometry>
         <material name="Grey"/>
@@ -281,5 +281,5 @@
         <origin xyz="0 0 -0.0005" rpy="0 0 0"/>
         <geometry>
-          <mesh filename="../meshes/iiwa7/collision/link_7.stl"/>
+          <mesh filename="package://kmr_iiwa_description/meshes/iiwa7/collision/link_7.stl"/>
         </geometry>
         <material name="Grey"/>

File: code/ros2_ws/src/kmr_iiwa_description/xacro/kmr_base.xacro (robot description, xacro)
@@ -17,7 +17,7 @@
   <xacro:property name="kmr_height" value="0.70"/> <!-- m, Z direction -->
   <xacro:property name="kmr_mesh_body"
-                   value="../meshes/kmr_base/kmr_base_body.stl"/>
+                   value="package://kmr_iiwa_description/meshes/kmr_base/kmr_base_body.stl"/>
   <xacro:property name="kmr_mesh_skirt"
-                   value="../meshes/kmr_base/kmr_base_skirt.stl"/>
+                   value="package://kmr_iiwa_description/meshes/kmr_base/kmr_base_skirt.stl"/>
   <!-- base_link -->
   <link name="base_link">

File: code/ros2_ws/src/kmr_iiwa_description/xacro/kmr_iiwa.urdf.xacro (robot description, xacro)
@@ -23,5 +23,5 @@
     <origin xyz="${iiwa_mount_x} ${iiwa_mount_y} ${iiwa_mount_z}" rpy="0 0 0"/>
   </xacro:iiwa7>
-  <xacro:kmr_gripper parent="iiwa_link_ee" mesh_path="../meshes/gripper">
+  <xacro:kmr_gripper parent="iiwa_link_ee" mesh_path="package://kmr_iiwa_description/meshes/gripper">
     <origin xyz="0 0 0" rpy="0 0 0"/>
   </xacro:kmr_gripper>
@@ -29,5 +29,5 @@
   <xacro:property name="camera_mount_y" value="0.184"/>
   <xacro:property name="camera_mount_z" value="${kmr_height}"/>
-  <xacro:kmr_camera_mount parent="base_link" mesh_path="../meshes/camera">
+  <xacro:kmr_camera_mount parent="base_link" mesh_path="package://kmr_iiwa_description/meshes/camera">
     <origin xyz="${camera_mount_x} ${camera_mount_y} ${camera_mount_z}" rpy="0 0 0"/>
   </xacro:kmr_camera_mount>

Commit message: added door collision, implemented accurate gripping of door handle

File: code/ros2_ws/src/kmr_iiwa_description/urdf/kmr_iiwa_full.urdf (robot description, URDF)
Before this commit: robot kmr_iiwa, 19 links, 18 joints
Joints:
- joint gripper_finger_1_joint: limit lower=0.0 upper=0.025 effort=30.0 velocity=0.1 -> lower=0.0 upper=0.026 effort=30.0 velocity=0.1
- joint gripper_finger_2_joint: limit lower=0.0 upper=0.025 effort=30.0 velocity=0.1 -> lower=0.0 upper=0.026 effort=30.0 velocity=0.1
- joint gripper_finger_3_joint: limit lower=0.0 upper=0.025 effort=30.0 velocity=0.1 -> lower=0.0 upper=0.026 effort=30.0 velocity=0.1
- joint gripper_finger_4_joint: limit lower=0.0 upper=0.025 effort=30.0 velocity=0.1 -> lower=0.0 upper=0.026 effort=30.0 velocity=0.1

Commit message: increased gripper finger max force

File: code/ros2_ws/src/kmr_iiwa_description/urdf/kmr_iiwa_full.urdf (robot description, URDF)
Before this commit: robot kmr_iiwa, 19 links, 18 joints
Joints:
- joint gripper_finger_1_joint: limit lower=0.0 upper=0.026 effort=30.0 velocity=0.1 -> lower=0.0 upper=0.026 effort=200.0 velocity=0.1
- joint gripper_finger_2_joint: limit lower=0.0 upper=0.026 effort=30.0 velocity=0.1 -> lower=0.0 upper=0.026 effort=200.0 velocity=0.1
- joint gripper_finger_3_joint: limit lower=0.0 upper=0.026 effort=30.0 velocity=0.1 -> lower=0.0 upper=0.026 effort=200.0 velocity=0.1
- joint gripper_finger_4_joint: limit lower=0.0 upper=0.026 effort=30.0 velocity=0.1 -> lower=0.0 upper=0.026 effort=200.0 velocity=0.1

File: code/ros2_ws/src/kmr_iiwa_description/xacro/gripper.xacro (robot description, xacro)
@@ -106,5 +106,5 @@
         <!-- os u lokalnom okviru prsta; +q = zatvaranje prema centru za sva 4 prsta -->
         <axis xyz="-1 0 0"/>
-        <limit lower="0.0" upper="0.026" effort="30.0" velocity="0.1"/>
+        <limit lower="0.0" upper="0.026" effort="200.0" velocity="0.1"/>
         <!-- damping se ionako pregazi actuator konfiguracijom u Isaac Labu -->
         <dynamics damping="10.0" friction="0.0"/>

Commit message: reverted to old gripper force

File: code/ros2_ws/src/kmr_iiwa_description/urdf/kmr_iiwa_full.urdf (robot description, URDF)
Before this commit: robot kmr_iiwa, 19 links, 18 joints
Joints:
- joint gripper_finger_1_joint: limit lower=0.0 upper=0.026 effort=200.0 velocity=0.1 -> lower=0.0 upper=0.026 effort=30.0 velocity=0.1
- joint gripper_finger_2_joint: limit lower=0.0 upper=0.026 effort=200.0 velocity=0.1 -> lower=0.0 upper=0.026 effort=30.0 velocity=0.1
- joint gripper_finger_3_joint: limit lower=0.0 upper=0.026 effort=200.0 velocity=0.1 -> lower=0.0 upper=0.026 effort=30.0 velocity=0.1
- joint gripper_finger_4_joint: limit lower=0.0 upper=0.026 effort=200.0 velocity=0.1 -> lower=0.0 upper=0.026 effort=30.0 velocity=0.1

File: code/ros2_ws/src/kmr_iiwa_description/xacro/gripper.xacro (robot description, xacro)
@@ -106,5 +106,5 @@
         <!-- os u lokalnom okviru prsta; +q = zatvaranje prema centru za sva 4 prsta -->
         <axis xyz="-1 0 0"/>
-        <limit lower="0.0" upper="0.026" effort="200.0" velocity="0.1"/>
+        <limit lower="0.0" upper="0.026" effort="30.0" velocity="0.1"/>
         <!-- damping se ionako pregazi actuator konfiguracijom u Isaac Labu -->
         <dynamics damping="10.0" friction="0.0"/>

Commit message: changed gripper force, stiffness and damping

File: code/ros2_ws/src/kmr_iiwa_description/urdf/kmr_iiwa_full.urdf (robot description, URDF)
Before this commit: robot kmr_iiwa, 19 links, 18 joints
Joints:
- joint gripper_finger_1_joint: limit lower=0.0 upper=0.026 effort=30.0 velocity=0.1 -> lower=0.0 upper=0.026 effort=600.0 velocity=0.1
- joint gripper_finger_2_joint: limit lower=0.0 upper=0.026 effort=30.0 velocity=0.1 -> lower=0.0 upper=0.026 effort=600.0 velocity=0.1
- joint gripper_finger_3_joint: limit lower=0.0 upper=0.026 effort=30.0 velocity=0.1 -> lower=0.0 upper=0.026 effort=600.0 velocity=0.1
- joint gripper_finger_4_joint: limit lower=0.0 upper=0.026 effort=30.0 velocity=0.1 -> lower=0.0 upper=0.026 effort=600.0 velocity=0.1

File: code/ros2_ws/src/kmr_iiwa_description/xacro/gripper.xacro (robot description, xacro)
@@ -106,5 +106,5 @@
         <!-- os u lokalnom okviru prsta; +q = zatvaranje prema centru za sva 4 prsta -->
         <axis xyz="-1 0 0"/>
-        <limit lower="0.0" upper="0.026" effort="30.0" velocity="0.1"/>
+        <limit lower="0.0" upper="0.026" effort="600.0" velocity="0.1"/>
         <!-- damping se ionako pregazi actuator konfiguracijom u Isaac Labu -->
         <dynamics damping="10.0" friction="0.0"/>

Commit message: fucked around, implemented lidar, walls and all sorts of stuff, revolute and sliding door work now

File: code/ros2_ws/src/kmr_iiwa_description/urdf/kmr_iiwa_full.urdf (robot description, URDF)
Before this commit: robot kmr_iiwa, 19 links, 18 joints
Links:
- added link lidar_link
Joints:
- added joint lidar_joint: type fixed, parent base_link, child lidar_link, origin xyz=0.5700000000000001 0.0 0.08 rpy=0 0 0

File: code/ros2_ws/src/kmr_iiwa_description/urdf/revolute_door.urdf (robot description, URDF)
Before this commit: robot revolute_door, 7 links, 6 joints
Links:
- added link wall_left, mass 100; collision box size=0.06 2.5 2.0; visual box size=0.06 2.5 2.0
- added link wall_right, mass 100; collision box size=0.06 2.5 2.0; visual box size=0.06 2.5 2.0
Joints:
- added joint wall_left_joint: type fixed, parent door_frame, child wall_left, origin xyz=0 0 0 rpy=0 0 0
- added joint wall_right_joint: type fixed, parent door_frame, child wall_right, origin xyz=0 0 0 rpy=0 0 0
- joint hinge_joint: limit lower=0.0 upper=1.57 effort=200 velocity=2.0 -> lower=0.0 upper=2.36 effort=200 velocity=2.0

File: code/ros2_ws/src/kmr_iiwa_description/urdf/sliding_door.urdf (robot description, URDF)
Before this commit: robot sliding_door, 6 links, 5 joints
Links:
- added link wall_left, mass 100; collision box size=0.06 2.5 2.0; visual box size=0.06 2.5 2.0
- added link wall_right, mass 100; collision box size=0.06 2.5 2.0; visual box size=0.06 2.5 2.0
Joints:
- added joint wall_left_joint: type fixed, parent slide_frame, child wall_left, origin xyz=0 0 0 rpy=0 0 0
- added joint wall_right_joint: type fixed, parent slide_frame, child wall_right, origin xyz=0 0 0 rpy=0 0 0
- joint slide_joint: limit lower=0.0 upper=0.8 effort=200 velocity=1.0 -> lower=0.0 upper=1.0 effort=200 velocity=1.0; origin xyz=0 0 0 rpy=0 0 0 -> xyz=0.07 0 0 rpy=0 0 0

File: code/ros2_ws/src/kmr_iiwa_description/xacro/kmr_iiwa.urdf.xacro (robot description, xacro)
@@ -6,4 +6,5 @@
   <xacro:include filename="gripper.xacro"/>
   <xacro:include filename="camera_mount.xacro"/>
+  <xacro:include filename="lidar_mount.xacro"/>
   <xacro:include filename="iiwa7.xacro"/>
   <xacro:include filename="kmr_iiwa_ros2_control.xacro"/>
@@ -32,4 +33,10 @@
     <origin xyz="${camera_mount_x} ${camera_mount_y} ${camera_mount_z}" rpy="0 0 0"/>
   </xacro:kmr_camera_mount>
+  <xacro:property name="lidar_mount_x" value="${kmr_length/2 + 0.03}"/>
+  <xacro:property name="lidar_mount_y" value="0.0"/>
+  <xacro:property name="lidar_mount_z" value="0.08"/>
+  <xacro:kmr_lidar_mount parent="base_link">
+    <origin xyz="${lidar_mount_x} ${lidar_mount_y} ${lidar_mount_z}" rpy="0 0 0"/>
+  </xacro:kmr_lidar_mount>
   <xacro:kmr_iiwa_ros2_control
       commands_topic="/isaac_joint_commands"
