Commit message: added walls to rl door urdfs, reconverted to usd

File: code/ros2_ws/src/kmr_iiwa_description/urdf/revolute_door_rl.urdf (robot description, URDF)
Before this commit: robot revolute_door_rl, 3 links, 2 joints
Links:
- added link wall_left, mass 100; collision box size=0.06 2.5 2.0; visual box size=0.06 2.5 2.0
- added link wall_right, mass 100; collision box size=0.06 2.5 2.0; visual box size=0.06 2.5 2.0
Joints:
- added joint wall_left_joint: type fixed, parent door_frame, child wall_left, origin xyz=0 0 0 rpy=0 0 0
- added joint wall_right_joint: type fixed, parent door_frame, child wall_right, origin xyz=0 0 0 rpy=0 0 0

File: code/ros2_ws/src/kmr_iiwa_description/urdf/sliding_door_rl.urdf (robot description, URDF)
Before this commit: robot sliding_door_rl, 3 links, 2 joints
Links:
- added link wall_left, mass 100; collision box size=0.06 2.5 2.0; visual box size=0.06 2.5 2.0
- added link wall_right, mass 100; collision box size=0.06 2.5 2.0; visual box size=0.06 2.5 2.0
Joints:
- added joint wall_left_joint: type fixed, parent door_frame, child wall_left, origin xyz=0 0 0 rpy=0 0 0
- added joint wall_right_joint: type fixed, parent door_frame, child wall_right, origin xyz=0 0 0 rpy=0 0 0

Commit message: increased revolute door hinge limit to 135 deg instead of 90 deg

File: code/ros2_ws/src/kmr_iiwa_description/urdf/revolute_door_rl.urdf (robot description, URDF)
Before this commit: robot revolute_door_rl, 5 links, 4 joints
Joints:
- joint door_dof_joint: limit lower=0.0 upper=1.57 effort=200 velocity=2.0 -> lower=0.0 upper=2.36 effort=200 velocity=2.0
