Commit message: updated to have same 1.0m range as model-based approach door

File: code/ros2_ws/src/kmr_iiwa_description/urdf/sliding_door_rl.urdf (robot description, URDF)
Before this commit: robot sliding_door_rl, 5 links, 4 joints
Joints:
- joint door_dof_joint: limit lower=0.0 upper=0.8 effort=200 velocity=1.0 -> lower=0.0 upper=1.0 effort=200 velocity=1.0
